File: klon/klon.brd (EAGLE design)
At the start: 160 x 100 mm, 8 parts, among them IC1 TL072P

Commit message: library tweaks.
Parts:
- added U$1: (no value), perfboards:9X7_CM
- added U$2: 2_1MM-JACK-PLUG, pedal-lilbrary:JACK-PLUG-2.1MM
- moved IC1 79.6 mm to (41.9, 69.8)
Connections:
- net +9V: now also U$2.P$1
- net GND: now also U$2.P$2
Routing:
- net +9V: track 0.00 -> 12.7 mm
- net GND: track 0.00 -> 5.08 mm
Changed lines of the file:
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@@
 <attribute name="VALUE" x="-72.4916" y="77.1398" size="1.27" layer="27" ratio="12"/>
 </element>
-<element name="IC1" library="linear" library_urn="urn:adsk.eagle:library:262" package="DIL08" package3d_urn="urn:adsk.eagle:package:16409/2" value="TL072P" x="-36.83" y="81.28" smashed="yes">
-<attribute name="NAME" x="-42.164" y="78.359" size="1.27" layer="25" ratio="10" rot="R90"/>
-<attribute name="POPULARITY" value="13" x="0" y="0" size="1.778" layer="27" display="off"/>
-<attribute name="VALUE" x="-40.386" y="80.645" size="1.27" layer="27" ratio="10"/>
+<element name="IC1" library="linear" library_urn="urn:adsk.eagle:library:262" package="DIL08" package3d_urn="urn:adsk.eagle:package:16409/2" value="TL072P" x="41.91" y="69.85" smashed="yes">
+<attribute name="NAME" x="36.576" y="66.929" size="1.27" layer="25" ratio="10" rot="R90"/>
+<attribute name="POPULARITY" value="13" x="78.74" y="-11.43" size="1.778" layer="27" display="off"/>
+<attribute name="VALUE" x="38.354" y="69.215" size="1.27" layer="27" ratio="10"/>
 </element>
 <element name="J1" library="mb-jacks" package="CLOSED_MONO_JACK" value="" x="-21.59" y="81.28" smashed="yes">
@@
 <attribute name="VALUE" x="-20.3106" y="88.9254" size="1.27" layer="27" ratio="12"/>
 </element>
+<element name="U$1" library="perfboards" package="9X7_CM" value="" x="25.4" y="10.16" smashed="yes">
+<attribute name="DEPTH" value="1.6mm" x="25.4" y="10.16" size="1.778" layer="27" display="off"/>
+<attribute name="HEIGHT" value="7cm" x="25.4" y="10.16" size="1.778" layer="27" display="off"/>
+<attribute name="HOLE_DIA" value="3.7mm" x="25.4" y="10.16" size="1.778" layer="27" display="off"/>
+<attribute name="PITCH" value="0.1in" x="25.4" y="10.16" size="1.778" layer="27" display="off"/>
+<attribute name="SIDES" value="2" x="25.4" y="10.16" size="1.778" layer="27" display="off"/>
+<attribute name="WIDTH" value="9cm" x="25.4" y="10.16" size="1.778" layer="27" display="off"/>
+</element>
+<element name="U$2" library="pedal-lilbrary" package="JACK-PLUG-2.1MM" value="2_1MM-JACK-PLUG" x="35.56" y="68.58" smashed="yes" rot="R90"/>
 </elements>
 <signals>
@@
 <signal name="GND">
 <contactref element="IC1" pad="8"/>
+<contactref element="U$2" pad="P$2"/>
+<wire x1="35.56" y1="71.12" x2="38.1" y2="71.12" width="1.27" layer="16"/>
+<wire x1="38.1" y1="71.12" x2="38.1" y2="73.66" width="1.27" layer="16"/>
 </signal>
 <signal name="+9V">
 <contactref element="IC1" pad="4"/>
+<contactref element="U$2" pad="P$1"/>
+<wire x1="35.56" y1="68.58" x2="45.72" y2="68.58" width="1.27" layer="16"/>
+<wire x1="45.72" y1="68.58" x2="45.72" y2="66.04" width="1.27" layer="16"/>
 </signal>
 <signal name="N$3">
 <contactref element="IC1" pad="3"/>
 <contactref element="C1" pad="2"/>
-<wire x1="-45.72" y1="80.01" x2="-35.56" y2="77.47" width="0" layer="19" extent="1-1"/>
+<wire x1="-45.72" y1="80.01" x2="43.18" y2="66.04" width="0" layer="19" extent="1-1"/>
 </signal>
 <signal name="N$4">
 <contactref element="IC1" pad="1"/>
 <contactref element="IC1" pad="2"/>
-<wire x1="-40.64" y1="77.47" x2="-38.1" y2="77.47" width="0" layer="19" extent="1-1"/>
+<wire x1="38.1" y1="66.04" x2="40.64" y2="66.04" width="0" layer="19" extent="1-1"/>
 </signal>
 </signals>
