File: klon/klon.brd.old2.brd (EAGLE design)
At the start: 160 x 100 mm, 64 parts, among them IC1 MAX1044, IC2 TL072P, IC3 TL072P

Commit message: Klon schematic
Parts:
- removed C10, C9: 68n, capacitor-wima:C10B5
- removed C11, C13, C18, C3, C4, C5: 1µ, pedal-library:C-E-0.1_0.15
- removed C12: 390p, pedal-library:C-C-0.1_0.05
- removed C14: 82n, pedal-library:C-PP-0.6_0.2
- removed C15: 2.2n, pedal-library:C-PP-0.4_0.15
- removed C16: 22n, pedal-library:C-PP-0.4_0.2
- removed C17: 4.7n, pedal-library:C-PP-0.4_0.2
- removed C19: 470p, pedal-library:C-C-0.1_0.05
- removed C20: 330p, pedal-library:C-C-0.1_0.05
- removed C21: 3.9n, pedal-library:C-PP-0.4_0.1
- removed C22: 4.7, pedal-library:C-E-0.1_0.15
- removed C7, C8: 0.1µ, capacitor-wima:C10B5
- removed D2, D3: 1N34A, diode:D-7.5
- removed IC2, IC3: TL072P, linear:DIL08
- removed LEVEL, TREBLE: 10kB, pedal-library:1X03
- removed R10, R18: 15k, pedal-library:0204/7
- removed R11: 422k, pedal-library:0204/7
- removed R12, R8: 1k, pedal-library:0204/7
- removed R13: 47k, pedal-library:0204/7
- removed R14: 22k, pedal-library:0204/7
- removed R15: 27k, pedal-library:0204/7
- removed R16: 12k, pedal-library:0204/7
- removed R17, R7: 1.5k, pedal-library:0204/7
- removed R19: 392K, pedal-library:0204/7
- removed R20, R22: 100k, pedal-library:0204/7
- removed R21: 1.8k, pedal-library:0204/7
- removed R23: 4.7k, pedal-library:0204/7
- removed R24: 560, pedal-library:0204/7
- removed R25, R26: 68K, pedal-library:0204/7
- removed R3, R5: 10k, pedal-library:0204/7
- removed R4: 1M, pedal-library:0204/7
- removed R6: 5.1k, pedal-library:0204/7
- removed R9: 2k, pedal-library:0204/7
- removed RV-GAIN: 100k, pedal-library:1X06
- removed S1: 3PDT9-PIN-HEADER, pedal-library:MA09-1
- removed U$5: INSTRUMENT-JACKPINS, pedal-library:1X03
- removed U$7: 330n, pedal-library:C-PP-0.6_0.15
- C1: value 47µ -> 47u
- C2: value 1µ -> (none)
- U$1: value 9x7 -> (none)
- moved D1 5.68 mm to (17.8, 47.0), flipped to the bottom
- moved U$2 5.68 mm to (15.2, 47.0), flipped to the bottom, turned to 90 degrees
- moved C1 5.68 mm to (20.3, 47.0)
- moved IC1 5.68 mm to (36.8, 44.5)
- moved U$4 5.68 mm to (25.4, 44.5)
- moved U$1 5.68 mm to (5.08, 7.62)
- moved R2 5.68 mm to (17.8, 38.1)
- moved C6 5.68 mm to (19.1, 40.6)
- moved R1 5.68 mm to (22.9, 43.2)
- moved U$3 5.68 mm to (29.2, 38.1)
- moved C2 2.54 mm to (26.7, 33.0)
Connections:
- removed net -8.6V: C4.+, IC1.5, IC3.4
- removed net N$1: C2.-, C3.+, IC1.2
- removed net N$10: C10.2, C8.1, IC2.1, IC2.2, R6.2
- removed net N$11: C10.1, R6.1, R7.2, RV-GAIN.5, U$7.2
- removed net N$12: R9.2, RV-GAIN.1
- removed net N$13: C14.1, R10.2, R9.1
- removed net N$14: C11.-, R12.1
- removed net N$15: C13.-, D2.C, D3.A, R12.2
- removed net N$16: C11.+, C12.1, IC2.7, R11.1
- removed net N$17: C12.2, C14.2, IC2.6, R10.1, R11.2
- removed net N$18: C13.+, C15.2, R13.1
- removed net N$19: C15.1, R14.2
- removed net N$2: C3.-, IC1.4
- removed net N$20: R14.1, R15.1, R16.1, RV-GAIN.6
- removed net N$21: C16.1, C17.1, R16.2
- removed net N$22: C16.2, C17.2, R15.2, R18.1
- removed net N$23: C18.+, R17.1, R18.2
- removed net N$24: R21.2, TREBLE.1
- removed net N$25: C19.2, C20.2, IC3.1, R19.2, R20.2, R21.1
- removed net N$26: C19.1, C20.1, IC3.2, R13.2, R19.1
- removed net N$27: C21.1, IC3.6, R20.1, TREBLE.2
- removed net N$28: C22.+, IC3.7, R22.1, R23.1
- removed net N$29: R23.2, TREBLE.3
- removed net N$30: C21.2, R22.2
- removed net N$31: C22.-, R24.2
- removed net N$32: LEVEL.3, R24.1
- removed net N$33: LEVEL.2, R26.1, S1.3
- removed net N$34: R25.1, S1.9
- removed net N$35: R25.2, R26.2, S1.6
- removed net N$4: C2.+, U$3.A, U$4.C
- removed net N$7: R8.2, U$7.1
- removed net N$8: C8.2, C9.1, R17.2, R5.1
- removed net N$9: C9.2, IC2.5, R5.2, RV-GAIN.2
- net +16.2V: no longer C5.+, IC3.8
- net +4.5V: no longer IC3.3, IC3.5, R7.1, R8.1, RV-GAIN.3, RV-GAIN.4
- net +9V: now also U$2.2; no longer IC2.8, U$2.1
- net GND: now also U$2.1; no longer C18.-, C4.-, C5.-, D2.A, D3.C, IC2.4, LEVEL.1, R4.1, U$2.2, U$5.1
- net N$3: now also U$3.A, U$4.C; no longer C7.1, R3.2
- net N$5: now also IC1.4; no longer R3.1, U$5.3
- net N$6: now also IC1.2; no longer C7.2, IC2.3, R4.2
Routing:
- net N$1: track 7.62 -> 0.00 mm
- net N$6: track 0.00 -> 5.08 mm
- net N$3: track 0.00 -> 5.08 mm
- net N$4: track 5.08 -> 0.00 mm
- net N$5: track 0.00 -> 2.54 mm
- net -8.6V: track 2.54 -> 0.00 mm
