File: reflow-oven/reflow-arduino-controller.sch (EAGLE design)
At the start: 3 parts, among them U1 ARGON

Commit message: Add encoder library.
Connections:
- new net ENC_A: U1.D2
- new net ENC_B: U1.SCK
- new net ENC_SWITCH: U1.D3
Changed lines of the file:
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@@
+</segment>
+</net>
+<net name="ENC_SWITCH" class="0">
+<segment>
+<pinref part="U1" gate="U1" pin="D3"/>
+<wire x1="104.14" y1="78.74" x2="134.62" y2="78.74" width="0.1524" layer="91"/>
+<label x="134.62" y="78.74" size="0.8128" layer="95" xref="yes"/>
+</segment>
+</net>
+<net name="ENC_A" class="0">
+<segment>
+<pinref part="U1" gate="U1" pin="D2"/>
+<wire x1="104.14" y1="76.2" x2="134.62" y2="76.2" width="0.1524" layer="91"/>
+<label x="134.62" y="76.2" size="0.8128" layer="95" xref="yes"/>
+</segment>
+</net>
+<net name="ENC_B" class="0">
+<segment>
+<pinref part="U1" gate="U1" pin="SCK"/>
+<wire x1="78.74" y1="83.82" x2="55.88" y2="83.82" width="0.1524" layer="91"/>
+<label x="55.88" y="83.82" size="0.8128" layer="95" rot="R180" xref="yes"/>
 </segment>
 </net>
